Commit message: Your descriptive commit message here

File: urdf/green_cylinder.urdf (robot description, URDF)
Before this commit: robot red_cylinder, 1 links, 0 joints
Links:
- link cylinder: mass 10 -> 20; geometry collision cylinder length=10 radius=1.0; visual cylinder length=10 radius=1.0

File: urdf/orange_cylinder.urdf (robot description, URDF)
Before this commit: robot red_cylinder, 1 links, 0 joints
Links:
- link cylinder: mass 10 -> 20; geometry collision cylinder length=10 radius=1.0; visual cylinder length=10 radius=1.0

File: urdf/red_cylinder.urdf (robot description, URDF)
Before this commit: robot red_cylinder, 1 links, 0 joints
Links:
- link cylinder: mass 10 -> 20; geometry collision cylinder length=10 radius=1.0; visual cylinder length=10 radius=1.0
